File: WiFi-Septic-Controller.sch (KiCad schematic (older format))
At the start: 99 parts, among them J1 Screw_Terminal_01x02, J2 Screw_Terminal_01x02, J3 Screw_Terminal_01x03, J4 Screw_Terminal_01x06, J5 USB_B_Micro, J6 GWT-C1627A-RGB, J7 Cortex Debug, J8 Screw_Terminal_01x03, Q1 2N7002, Q2 2N7002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

Commit message: Changed ALM label on schematic to match PCB silkscreen.
Other:
- note added: "AL"
- note removed: "ALM"
Changed lines of the file:
@@
 P2
 Text Notes 14950 3200 0    60   ~ 0
-ALM
+AL
 Text Notes 14950 3300 0    60   ~ 0
 S1

Commit message: Changed transformer part number. Alarm Labels on schematic now match PCB positions. Update PCB Status.
Parts:
- T1: Vendor Part Number 553-VPP20-250 -> 553-VPP16-310
Other:
- note added: "Air Pump\nAlarm"
- note removed: "Air Compressor\nAlarm"
Changed lines of the file:
@@
 F 5 "VPP20-250" H 3000 2050 50  0001 C CNN "Part Number"
 F 6 "Mouser" H 3000 2050 50  0001 C CNN "Vendor"
-F 7 "553-VPP20-250" H 3000 2050 50  0001 C CNN "Vendor Part Number"
+F 7 "553-VPP16-310" H 3000 2050 50  0001 C CNN "Vendor Part Number"
 	1    3000 2050
 	1    0    0    -1
@@
 Text Notes 15150 3200 0    60   ~ 0
 - Alarm Output
-Text Notes 14950 5200 0    60   ~ 0
+Text Notes 14950 5750 0    60   ~ 0
 AA1
-Text Notes 15200 5200 0    60   ~ 0
+Text Notes 15200 5750 0    60   ~ 0
 - Air Alarm
-Text Notes 14950 5300 0    60   ~ 0
+Text Notes 14950 5650 0    60   ~ 0
 AA2
-Text Notes 15200 5300 0    60   ~ 0
+Text Notes 15200 5650 0    60   ~ 0
 - Air Alarm
-Text Notes 14950 5400 0    60   ~ 0
+Text Notes 14950 5550 0    60   ~ 0
 FA1
-Text Notes 15200 5400 0    60   ~ 0
+Text Notes 15200 5550 0    60   ~ 0
 - Float Alarm
-Text Notes 14950 5500 0    60   ~ 0
+Text Notes 14950 5450 0    60   ~ 0
 FA2
-Text Notes 15200 5500 0    60   ~ 0
+Text Notes 15200 5450 0    60   ~ 0
 - Float Alarm
-Text Notes 14950 5600 0    60   ~ 0
+Text Notes 14950 5350 0    60   ~ 0
 BA1
-Text Notes 15200 5600 0    60   ~ 0
+Text Notes 15200 5350 0    60   ~ 0
 - Bleach Alarm
-Text Notes 14950 5700 0    60   ~ 0
+Text Notes 14950 5250 0    60   ~ 0
 BA2
-Text Notes 15200 5700 0    60   ~ 0
+Text Notes 15200 5250 0    60   ~ 0
 - Bleach Alarm
 Wire Wire Line
@@
 $EndComp
 Text Notes 10950 5150 0    75   Italic 15
-Air Compressor\nAlarm
+Bleach Level\nAlarm
 $Comp
 L power:VCC #PWR0101
@@
 Tank High Float\nAlarm
 Text Notes 10950 6250 0    75   Italic 15
-Bleach Level\nAlarm
+Air Pump\nAlarm
 Text Notes 11150 3750 2    60   ~ 0
 10mA

Commit message: Change alarm input resistors
The 100k alarm input resistors may be a high enough impedance to allow noise to trigger the over full alarm. Changed the resistors to 22k. Minor update to README file.
Parts:
- R13, R14, R15, R16, R17, R18: value 100k -> 22k; Part Number ERJ-P08J104V -> ERJ-P08J223V; Vendor Part Number 667-ERJ-P08J104V -> 667-ERJ-P08J223V
Changed lines of the file:
@@
 P 12850 5200
 F 0 "R14" V 12950 5200 50  0000 C CNN
-F 1 "100k" V 12850 5200 50  0000 C CNN
+F 1 "22k" V 12850 5200 50  0000 C CNN
 F 2 "Resistors_SMD:R_1206" V 12780 5200 50  0001 C CNN
 F 3 "" V 12850 5200 50  0001 C CNN
 F 4 "Panasonic" H 12850 5200 60  0001 C CNN "Manufacturer"
-F 5 "ERJ-P08J104V" H 12850 5200 60  0001 C CNN "Part Number"
+F 5 "ERJ-P08J223V" H 12850 5200 60  0001 C CNN "Part Number"
 F 6 "Mouser" H 12850 5200 60  0001 C CNN "Vendor"
-F 7 "667-ERJ-P08J104V" H 12850 5200 60  0001 C CNN "Vendor Part Number"
+F 7 "667-ERJ-P08J223V" H 12850 5200 60  0001 C CNN "Vendor Part Number"
 F 8 "5%" H 12900 5150 50  0001 L CNN "Tolerance"
 	1    12850 5200
@@
 P 12850 5800
 F 0 "R15" V 12950 5800 50  0000 C CNN
-F 1 "100k" V 12850 5800 50  0000 C CNN
+F 1 "22k" V 12850 5800 50  0000 C CNN
 F 2 "Resistors_SMD:R_1206" V 12780 5800 50  0001 C CNN
 F 3 "" V 12850 5800 50  0001 C CNN
 F 4 "Panasonic" H 12850 5800 60  0001 C CNN "Manufacturer"
-F 5 "ERJ-P08J104V" H 12850 5800 60  0001 C CNN "Part Number"
+F 5 "ERJ-P08J223V" H 12850 5800 60  0001 C CNN "Part Number"
 F 6 "Mouser" H 12850 5800 60  0001 C CNN "Vendor"
-F 7 "667-ERJ-P08J104V" H 12850 5800 60  0001 C CNN "Vendor Part Number"
+F 7 "667-ERJ-P08J223V" H 12850 5800 60  0001 C CNN "Vendor Part Number"
 F 8 "5%" H 12900 5750 50  0001 L CNN "Tolerance"
 	1    12850 5800
@@
 P 13350 5000
 F 0 "R13" V 13250 5000 50  0000 C CNN
-F 1 "100k" V 13350 5000 50  0000 C CNN
+F 1 "22k" V 13350 5000 50  0000 C CNN
 F 2 "Resistors_SMD:R_1206" V 13280 5000 50  0001 C CNN
 F 3 "" V 13350 5000 50  0001 C CNN
 F 4 "Panasonic" H 13350 5000 60  0001 C CNN "Manufacturer"
-F 5 "ERJ-P08J104V" H 13350 5000 60  0001 C CNN "Part Number"
+F 5 "ERJ-P08J223V" H 13350 5000 60  0001 C CNN "Part Number"
 F 6 "Mouser" H 13350 5000 60  0001 C CNN "Vendor"
-F 7 "667-ERJ-P08J104V" H 13350 5000 60  0001 C CNN "Vendor Part Number"
+F 7 "667-ERJ-P08J223V" H 13350 5000 60  0001 C CNN "Vendor Part Number"
 F 8 "5%" H 13400 4950 50  0001 L CNN "Tolerance"
 	1    13350 5000
@@
 P 13350 6000
 F 0 "R16" V 13250 6000 50  0000 C CNN
-F 1 "100k" V 13350 6000 50  0000 C CNN
+F 1 "22k" V 13350 6000 50  0000 C CNN
 F 2 "Resistors_SMD:R_1206" V 13280 6000 50  0001 C CNN
 F 3 "" V 13350 6000 50  0001 C CNN
 F 4 "Panasonic" H 13350 6000 60  0001 C CNN "Manufacturer"
-F 5 "ERJ-P08J104V" H 13350 6000 60  0001 C CNN "Part Number"
+F 5 "ERJ-P08J223V" H 13350 6000 60  0001 C CNN "Part Number"
 F 6 "Mouser" H 13350 6000 60  0001 C CNN "Vendor"
-F 7 "667-ERJ-P08J104V" H 13350 6000 60  0001 C CNN "Vendor Part Number"
+F 7 "667-ERJ-P08J223V" H 13350 6000 60  0001 C CNN "Vendor Part Number"
 F 8 "5%" H 13400 5950 50  0001 L CNN "Tolerance"
 	1    13350 6000
@@
 P 12850 6300
 F 0 "R18" V 12950 6300 50  0000 C CNN
-F 1 "100k" V 12850 6300 50  0000 C CNN
+F 1 "22k" V 12850 6300 50  0000 C CNN
 F 2 "Resistors_SMD:R_1206" V 12780 6300 50  0001 C CNN
 F 3 "" V 12850 6300 50  0001 C CNN
 F 4 "Panasonic" H 12850 6300 60  0001 C CNN "Manufacturer"
-F 5 "ERJ-P08J104V" H 12850 6300 60  0001 C CNN "Part Number"
+F 5 "ERJ-P08J223V" H 12850 6300 60  0001 C CNN "Part Number"
 F 6 "Mouser" H 12850 6300 60  0001 C CNN "Vendor"
-F 7 "667-ERJ-P08J104V" H 12850 6300 60  0001 C CNN "Vendor Part Number"
+F 7 "667-ERJ-P08J223V" H 12850 6300 60  0001 C CNN "Vendor Part Number"
 F 8 "5%" H 12900 6250 50  0001 L CNN "Tolerance"
 	1    12850 6300
@@
 P 13350 6100
 F 0 "R17" V 13250 6100 50  0000 C CNN
-F 1 "100k" V 13350 6100 50  0000 C CNN
+F 1 "22k" V 13350 6100 50  0000 C CNN
 F 2 "Resistors_SMD:R_1206" V 13280 6100 50  0001 C CNN
 F 3 "" V 13350 6100 50  0001 C CNN
 F 4 "Panasonic" H 13350 6100 60  0001 C CNN "Manufacturer"
-F 5 "ERJ-P08J104V" H 13350 6100 60  0001 C CNN "Part Number"
+F 5 "ERJ-P08J223V" H 13350 6100 60  0001 C CNN "Part Number"
 F 6 "Mouser" H 13350 6100 60  0001 C CNN "Vendor"
-F 7 "667-ERJ-P08J104V" H 13350 6100 60  0001 C CNN "Vendor Part Number"
+F 7 "667-ERJ-P08J223V" H 13350 6100 60  0001 C CNN "Vendor Part Number"
 F 8 "5%" H 13400 6050 50  0001 L CNN "Tolerance"
 	1    13350 6100

Commit message: Update to KiCad 5.1 libraries.
Also updated custom libraries.
Parts:
- C1, C2: footprint Capacitors_SMD:CP_Elec_10x10.5 -> Capacitor_SMD:CP_Elec_10x10.5; symbol device:CP_Small -> Device:CP_Small
- C10, C17, C3, C5, C8: footprint Capacitors_SMD:C_0805 -> Capacitor_SMD:C_0805_2012Metric; symbol device:C_Small -> Device:C_Small
- C11, C12, C13, C14, C15, C16, C18, C19, C20, C21, C22, C4, C6, C7, C9: footprint Capacitors_SMD:C_0603 -> Capacitor_SMD:C_0603_1608Metric; symbol device:C_Small -> Device:C_Small
- D1: footprint Diodes_SMD:D_PowerDI-123 -> Diode_SMD:D_PowerDI-123; symbol device:D_Schottky_ALT -> Device:D_Schottky_ALT
- D10, D7, D8, D9: footprint LEDs:LED_0603 -> LED_SMD:LED_0603_1608Metric; symbol device:LED_ALT -> Device:LED_ALT
- D2: footprint Diodes_SMD:Diode_Bridge_DFS -> Diode_SMD:Diode_Bridge_Vishay_DFS; symbol device:D_Bridge_+-AA -> Device:D_Bridge_+-AA
- D3, D4, D5: footprint TO_SOT_Packages_SMD:SOT-23 -> Package_TO_SOT_SMD:SOT-23; symbol ti-ml:TPD2E2U06-Q1 -> Power_Protection-ML:TPD2E2U06
- D6: footprint TO_SOT_Packages_SMD:SOT-143 -> Package_TO_SOT_SMD:SOT-143; symbol ESD_Protection:PRTR5V0U2X -> Power_Protection-ML:PRTR5V0U2X
- J1: footprint TerminalBlock_Phoenix:TerminalBlock_Phoenix_PT-3.5mm_2pol -> TerminalBlock_Phoenix:TerminalBlock_Phoenix_PT-1,5-2-3.5-H_1x02_P3.50mm_Horizontal
- J3: footprint TerminalBlock_Phoenix:TerminalBlock_Phoenix_PT-3.5mm_3pol -> TerminalBlock_Phoenix:TerminalBlock_Phoenix_PT-1,5-3-3.5-H_1x03_P3.50mm_Horizontal
- J4: footprint TerminalBlock_Phoenix:TerminalBlock_Phoenix_PT-3.5mm_6pol -> TerminalBlock_Phoenix:TerminalBlock_Phoenix_PT-1,5-6-3.5-H_1x06_P3.50mm_Horizontal
- J5: footprint Connectors_USB:USB_Micro-B_Wuerth-614105150721_Vertical_CircularHoles -> Connector_USB:USB_Micro-B_Wuerth_614105150721_Vertical_CircularHoles
- J6: footprint adafruit-ml:GWT-C1627A-RGB -> Adafruit-ML:GWT-C1627A-RGB; symbol adafruit-ml:GWT-C1627A-RGB -> Adafruit-ML:GWT-C1627A-RGB
- J7: footprint Pin_Headers:Pin_Header_Straight_2x05_Pitch1.27mm_SMD -> Connector_PinHeader_1.27mm:PinHeader_2x05_P1.27mm_Vertical_SMD; symbol Connector:Conn_02x05_Odd_Even -> Connector_Generic:Conn_02x05_Odd_Even
- L1, L2: footprint Inductors_SMD:L_1206 -> Inductor_SMD:L_1206_3216Metric; symbol device:Ferrite_Bead -> Device:Ferrite_Bead
- L3: footprint Inductors_SMD:L_0603 -> Inductor_SMD:L_0603_1608Metric; symbol device:Ferrite_Bead -> Device:Ferrite_Bead
- MK1: footprint holes-ml:6-32_PTH_Mounting_Hole -> MountingHole-ML:6-32_PTH_Mounting_Hole; symbol Mechanical:Mounting_Hole_PAD -> Mechanical:MountingHole_Pad
- Q1, Q2, Q5, Q6, Q7, Q8, Q9: footprint TO_SOT_Packages_SMD:SOT-23 -> Package_TO_SOT_SMD:SOT-23; symbol Transistor:2N7002 -> Transistor_FET:2N7002
- Q3: footprint TO_SOT_Packages_SMD:SOT-23 -> Package_TO_SOT_SMD:SOT-23; symbol diodes-inc-ml:DMG2305UX -> Transistor_FET-ML:DMG2305UX
- Q4: footprint TO_SOT_Packages_SMD:SOT-363_SC-70-6 -> Package_TO_SOT_SMD:SOT-363_SC-70-6; symbol diodes-inc-ml:BCM857BS -> Transistor_BJT-ML:BCM857BS
- R1, R10, R11, R19, R2, R20, R21, R22, R23, R24, R25, R26, R28, R29, R3, R4, R5, R7, R8, R9: footprint Resistors_SMD:R_0603 -> Resistor_SMD:R_0603_1608Metric; symbol device:R -> Device:R
- R12, R13, R14, R15, R16, R17, R18, R6: footprint Resistors_SMD:R_1206 -> Resistor_SMD:R_1206_3216Metric; symbol device:R -> Device:R
- RL1, RL2: footprint ixys-ml:SIP-4 -> Relay_THT-ML:Relay_IXYS_PowerSIP; symbol ixys-ml:CPC1511Y -> Relay_SolidState-ML:CPC1511Y
- RV1: footprint Potentiometers:Potentiometer_Trimmer_Bourns_3339P_Horizontal -> Potentiometer_THT:Potentiometer_Bourns_3339P_Vertical; symbol device:POT -> Device:R_POT
- SW1: footprint Buttons_Switches_SMD:SW_SPST_B3U-1000P -> Button_Switch_SMD:SW_SPST_B3U-1000P
- SW2: footprint Buttons_Switches_SMD:SW_SPST_PTS645 -> Button_Switch_SMD:SW_SPST_PTS645
- T1: footprint triad-ml:VPP -> Transformer_THT-ML:Triad_VPP_5.0VA; symbol triad-ml:VPP-XFMR -> Transformer-ML:Triad_VPP20-250; Part Number VPP20-250 -> VPP16-310
- TP1, TP2: footprint Connectors_TestPoints:Test_Point_Pad_1.0x1.0mm -> TestPoint:TestPoint_THTPad_2.0x2.0mm_Drill1.0mm; symbol Connector:Test_Point_Flag -> Connector:TestPoint_Flag
- TP3: footprint Connectors_TestPoints:Test_Point_Keystone_5010-5014_Multipurpose -> TestPoint:TestPoint_Keystone_5010-5014_Multipurpose; symbol Connector:Test_Point_Flag -> Connector:TestPoint_Flag
- U1, U2: footprint ti-ml:SIL0008E -> Converter_DCDC-ML:Converter_DCDC_Texas-SIL0008E; symbol ti-ml:LMZ21700 -> Converter_DCDC-ML:LMZ21700
- U3, U4: footprint Housings_DIP:SMDIP-8_W9.53mm -> Package_DIP:SMDIP-8_W9.53mm; symbol onsemi-ml:MID400 -> Isolator-ML:MID400
- U5, U7: footprint TO_SOT_Packages_SMD:SOT-23-6 -> Package_TO_SOT_SMD:SOT-23-6; symbol Logic_74xgxx:74LVC2G14 -> 74xGxx:74LVC2G14
- U6: footprint atmel-ml:ATWINC1500-MR210XB -> RF_Module-ML:Microchip_ATWINC1500-MR210UB; symbol atmel-ml:ATWINC1500-MR210UB -> RF_WiFi-ML:ATWINC1500-MR210UB
- U8: footprint Housings_DFN_QFN:QFN-48-1EP_7x7mm_Pitch0.5mm -> Package_DFN_QFN:QFN-48-1EP_7x7mm_P0.5mm_EP5.15x5.15mm; symbol atmel-ml:SAMD21G18-M -> MCU_Microchip_SAMD-ML:SAMD21G18-M
- Y1: footprint abracon-ml:ABS07 -> Crystal-ML:Crystal_SMD_Abracon_ABS07-2Pin_3.2x1.5mm; symbol device:Crystal -> Device:Crystal
Other:
- note added: "Pump\nRelay"
- note added: "Pump\nSense"
- note added: "The SAMD21G18 does not have extra filtering on the analog power supply so analog measurements may not be ideal."
- note removed: "Effluent\nPump\nRelay"
- note removed: "Effluent\nPump\nSense"
- note removed: "The SAMD21G18 does not have extra filtering on the analog power supply so analog measurements may be ideal."

Commit message: Cleanup BOM. VCC now +3V3.
Add KiBoM support.
Cleanup part information in schematic.
Added power pins to schematic on multi-unit gates.
Parts:
- C1, C2: Description (none) -> CAP, SMD 10X10.5, 20%, EC, 50V
- C10, C5: Description (none) -> CAP, 0805, 22uf, 20%, X5R, 25V; Vendor Part Number 810-C2012X5R1A226M-3 -> 963-TMK212BBJ226MGTT
- C11, C12, C13, C14, C15, C22: Description (none) -> CAP, 0603, 0.1uF, 20%, X7R, 10V
- C16, C18: Description (none) -> CAP, 0603, 1uF, 20%, X7R, 10V
- C17, C3, C8: Description (none) -> CAP, 0805, 22uf, 20%, X5R, 25V
- C19, C20: Description (none) -> CAP, 0603, 15pF, 5%, C0G, 50V
- C21: Description (none) -> CAP, 0603, 0.1uF, 20%, X7R, 10V; Vendor Part Number 963-TMK212BBJ226MGTT -> 77-VJ0603Y104JXQPBC
- C4, C9: value 3.3nF -> 3300pF; Description (none) -> CAP, 0603, 3300pF, 5%, X7R, 10V
- C6, C7: value 1nF -> 1000pF; Description (none) -> CAP, 0603, 1000pF, 10%, X7R, 10V
- D1: Description (none) -> DIO, PowerDI123, Schottky Rectifier, 30V, 1A
- D10: Description (none) -> LED, 0603, Blue LED
- D2: Description (none) -> DIO, DFS, Bridge Diode, 2A, 600V
- D3, D4, D5: Description (none) -> TVS, SOT23, ESD TVS Protection, Dual
- D6: Description (none) -> TVS, SOT23, ESD Protection, USB
- D7: Description (none) -> LED, 0603, Yellow LED
- D8: Description (none) -> LED, 0603, Green LED
- D9: Description (none) -> LED, 0603, Red LED
- J1: Description (none) -> CON, THT, Terminal Block, 3.5mm, 2 Pos
- J2: footprint TerminalBlock_Phoenix:TerminalBlock_Phoenix_PT-3.5mm_2pol -> TerminalBlock_Phoenix:TerminalBlock_Phoenix_PT-1,5-2-3.5-H_1x02_P3.50mm_Horizontal; Description (none) -> CON, THT, Terminal Block, 3.5mm, 2 Pos
- J3: Description (none) -> CON, THT, Terminal Block, 3.5mm, 3 Pos
- J4: Description (none) -> CON, THT, Terminal Block, 3.5mm, 6 Pos
- J5: Description (none) -> CON, THT, Micro USB 2.0 Type AB, Vertical
- J6: Description (none) -> CON, THT, 2.54mm Socket, Single Row, Vertical, 18 Pos; Manufacturer (none) -> Samtec; Part Number (none) -> SSW-150-01-G-S; Vendor (none) -> Digikey; Vendor Part Number (none) -> SAM1209-50-ND
- J7: Description (none) -> CON, SMD, 1.27mm Header, Dual Row, Vertical, 10 Pos
- J8: footprint TerminalBlock_Phoenix:TerminalBlock_Phoenix_PT-3.5mm_3pol -> TerminalBlock_Phoenix:TerminalBlock_Phoenix_PT-1,5-3-3.5-H_1x03_P3.50mm_Horizontal; Description (none) -> CON, THT, Terminal Block, 3.5mm, 3 Pos
- L1, L2: value 1k@1MHz -> 1k@100MHz; Description (none) -> BEAD, 1206, 1k@100MHz, 2A
- L3: value 470@1MHz -> 470@100MHz; Description (none) -> BEAD, 0603, 470R@100MHz, 1A
- MK1, TP1, TP2: Notes (none) -> DNF
- Q1, Q2, Q5, Q6, Q7, Q8, Q9: Description (none) -> TRANS, SOT23, Mosfet, P-CH, 115mA, 60V
- Q3: Description (none) -> TRANS, SOT23, Mosfet, P-CH, -5A, -20V
- Q4: Description (none) -> TRANS, SOT363, Bipolar, PNP, Dual Matched
- R1: Description (none) -> RES, 0603, 1.21M, 1%, T100
- R10: Description (none) -> RES, 0603, 47k, 1%, T100
- R11, R24, R26, R3, R5, R9: Description (none) -> RES, 0603, 10k, 1%, T100
- R12, R13, R14, R15, R16, R17, R18, R6: Description (none) -> RES, 1206, 22k, 5%, T200
- R19, R20, R21: value 130 -> 130R; Description (none) -> RES, 0603, 130R, 1%, T100
- R2: Description (none) -> RES, 0603, 383k, 1%, T100
- R22: Description (none) -> RES, 0603, 4.7k, 1%, T100
- R23: value 39 -> 39R; Description (none) -> RES, 0603, 39R, 1%, T100
- R25: value 330 -> 330R; Description (none) -> RES, 0603, 330R, 1%, T100
- R28, R29: value 698 -> 698R; Description (none) -> RES, 0603, 698R, 1%, T100
- R4: value 169 -> 169R; Description (none) -> RES, 0603, 169R, 1%, T100
- R7: Description (none) -> RES, 0603, 232k, 1%, T100
- R8: Description (none) -> RES, 0603, 44.2k, 1%, T100
- RL1, RL2: Description (none) -> RLY, THT, Solid State, Form A, Protected, 230V, 450mA
- RV1: Description (none) -> POT, THT, 10k, Round
- SW1, SW2: Description (none) -> SW, SMD, Push Button
- T1: Description (none) -> XFMR, THT, 120/240V to 8/16V, 310mA
- U1, U2: Description (none) -> MODULE, SMD, Simple Switcher, 17V, .65A
- U3, U4: Description (none) -> IC, SMDIP8, Optical AC Line Monitor
- U5, U7: Description (none) -> IC, SOT23-6, Dual inverting Schmitt trigger
- U6: Description (none) -> MODULE, SMD, WiFi, u.FL connector
- U8: Description (none) -> IC, QFN44, MCU, ARM, 256kB Flash, 32kB SRAM, 48MHz
- Y1: Description (none) -> XTL, SMD, 32.768kHz
Connections:
- net VCC renamed +3V3
